File: KiCad Project/Data Mode Radio Cable.kicad_sch (KiCad schematic)
At the start: 11 parts, among them J1 TRRS, J2 2.5mm, J3 3.5mm, J4 RS232, SW1 PTT_LOCK, T1 600R, U1 PC817

Commit message: Add files via upload
Replaced project files with ones pointing to new per-project footprints
Parts:
- J1: footprint Keebio-Parts:TRRS-PJ-320A -> Library:TRRS-PJ-320A
- SW1: footprint Custom_Footprints:SPDT_Right_Angled_Switch -> Library:SPDT_Right_Angled_Switch
- T1: footprint Custom_Footprints:1-1_Audio_Transformer_600_ohm -> Library:1-1_Audio_Transformer_600_ohm
Changed lines of the file:
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@@
     (property "Reference" "T1" (id 0) (at 107.95 47.4726 0))
     (property "Value" "600R" (id 1) (at 107.95 49.784 0))
-    (property "Footprint" "Custom_Footprints:1-1_Audio_Transformer_600_ohm" (id 2) (at 107.95 57.15 0)
+    (property "Footprint" "Library:1-1_Audio_Transformer_600_ohm" (id 2) (at 107.95 57.15 0)
       (effects (font (size 1.27 1.27)) hide)
     )
@@
       (effects (font (size 1.27 1.27)) (justify left))
     )
-    (property "Footprint" "Keebio-Parts:TRRS-PJ-320A" (id 2) (at 40.64 44.45 0)
+    (property "Footprint" "Library:TRRS-PJ-320A" (id 2) (at 40.64 44.45 0)
       (effects (font (size 1.27 1.27)) hide)
     )
@@
     (property "Reference" "SW1" (id 0) (at 124.46 73.66 0))
     (property "Value" "PTT_LOCK" (id 1) (at 124.46 76.2 0))
-    (property "Footprint" "Custom_Footprints:SPDT_Right_Angled_Switch" (id 2) (at 124.46 81.28 0)
+    (property "Footprint" "Library:SPDT_Right_Angled_Switch" (id 2) (at 124.46 81.28 0)
       (effects (font (size 1.27 1.27)) hide)
     )
@@
     )
     (path "/00000000-0000-0000-0000-00005ffd1205"
-      (reference "J1") (unit 1) (value "TRRS") (footprint "Keebio-Parts:TRRS-PJ-320A")
+      (reference "J1") (unit 1) (value "TRRS") (footprint "Library:TRRS-PJ-320A")
     )
     (path "/00000000-0000-0000-0000-00005ffd8cb7"
@@
     )
     (path "/00000000-0000-0000-0000-000060350a0e"
-      (reference "SW1") (unit 1) (value "PTT_LOCK") (footprint "Custom_Footprints:SPDT_Right_Angled_Switch")
+      (reference "SW1") (unit 1) (value "PTT_LOCK") (footprint "Library:SPDT_Right_Angled_Switch")
     )
     (path "/00000000-0000-0000-0000-00005ffcb4e8"
-      (reference "T1") (unit 1) (value "600R") (footprint "Custom_Footprints:1-1_Audio_Transformer_600_ohm")
+      (reference "T1") (unit 1) (value "600R") (footprint "Library:1-1_Audio_Transformer_600_ohm")
     )
     (path "/00000000-0000-0000-0000-00005ffcdae6"
